File: Hardware/_autosave-rgb-strip.kicad_pcb (KiCad board)
At the start: 2 copper layers, 16 parts, among them CON1 BARREL_JACK, IC1 ATTINY84-P, P1 Bluetooth_Header, P2 CONN_01X03, Q1 HC49, SW1 SW_PUSH, U1 LM7805

Commit message: Created pcb layout
Parts:
- added P3: CONN_01X01, Pin_Headers:Pin_Header_Straight_1x01, B.Cu at (66.0, 77.5)
- added P4: CONN_01X01, Pin_Headers:Pin_Header_Straight_1x01, B.Cu at (81.3, 77.5)
Changed lines of the file:
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@@
 (kicad_pcb (version 4) (host pcbnew 4.0.0-2.201511301921+6191~38~ubuntu15.10.1-stable)
   (general
-    (links 35)
+    (links 37)
     (no_connects 1)
     (area 0 0 0 0)
@@
     (tracks 80)
     (zones 0)
-    (modules 16)
+    (modules 18)
     (nets 19)
   )
@@
       (net 1 GND))
   )
+  (module Pin_Headers:Pin_Header_Straight_1x01 (layer B.Cu)
+    (at 66.04 77.47)
+    (descr "Through hole pin header")
+    (tags "pin header")
+    (fp_text reference P3 (at 0 5.1) (layer B.SilkS)
+      (effects (font (size 1 1) (thickness 0.15)) (justify mirror))
+    )
+    (fp_text value CONN_01X01 (at 0 3.1) (layer B.Fab)
+      (effects (font (size 1 1) (thickness 0.15)) (justify mirror))
+    )
+    (fp_line (start 1.55 1.55) (end 1.55 0) (layer B.SilkS) (width 0.15))
+    (fp_line (start -1.75 1.75) (end -1.75 -1.75) (layer B.CrtYd) (width 0.05))
+    (fp_line (start 1.75 1.75) (end 1.75 -1.75) (layer B.CrtYd) (width 0.05))
+    (fp_line (start -1.75 1.75) (end 1.75 1.75) (layer B.CrtYd) (width 0.05))
+    (fp_line (start -1.75 -1.75) (end 1.75 -1.75) (layer B.CrtYd) (width 0.05))
+    (fp_line (start -1.55 0) (end -1.55 1.55) (layer B.SilkS) (width 0.15))
+    (fp_line (start -1.55 1.55) (end 1.55 1.55) (layer B.SilkS) (width 0.15))
+    (fp_line (start -1.27 -1.27) (end 1.27 -1.27) (layer B.SilkS) (width 0.15))
+    (pad 1 thru_hole rect (at 0 0) (size 2.2352 2.2352) (drill 1.016) (layers *.Cu *.Mask B.SilkS)
+      (net 1 GND))
+    (model Pin_Headers.3dshapes/Pin_Header_Straight_1x01.wrl
+      (at (xyz 0 0 0))
+      (scale (xyz 1 1 1))
+      (rotate (xyz 0 0 90))
+    )
+  )
+  (module Pin_Headers:Pin_Header_Straight_1x01 (layer B.Cu)
+    (at 81.28 77.47)
+    (descr "Through hole pin header")
+    (tags "pin header")
+    (fp_text reference P4 (at 0 5.1) (layer B.SilkS)
+      (effects (font (size 1 1) (thickness 0.15)) (justify mirror))
+    )
+    (fp_text value CONN_01X01 (at 0 3.1) (layer B.Fab)
+      (effects (font (size 1 1) (thickness 0.15)) (justify mirror))
+    )
+    (fp_line (start 1.55 1.55) (end 1.55 0) (layer B.SilkS) (width 0.15))
+    (fp_line (start -1.75 1.75) (end -1.75 -1.75) (layer B.CrtYd) (width 0.05))
+    (fp_line (start 1.75 1.75) (end 1.75 -1.75) (layer B.CrtYd) (width 0.05))
+    (fp_line (start -1.75 1.75) (end 1.75 1.75) (layer B.CrtYd) (width 0.05))
+    (fp_line (start -1.75 -1.75) (end 1.75 -1.75) (layer B.CrtYd) (width 0.05))
+    (fp_line (start -1.55 0) (end -1.55 1.55) (layer B.SilkS) (width 0.15))
+    (fp_line (start -1.55 1.55) (end 1.55 1.55) (layer B.SilkS) (width 0.15))
+    (fp_line (start -1.27 -1.27) (end 1.27 -1.27) (layer B.SilkS) (width 0.15))
+    (pad 1 thru_hole rect (at 0 0) (size 2.2352 2.2352) (drill 1.016) (layers *.Cu *.Mask B.SilkS)
+      (net 1 GND))
+    (model Pin_Headers.3dshapes/Pin_Header_Straight_1x01.wrl
+      (at (xyz 0 0 0))
+      (scale (xyz 1 1 1))
+      (rotate (xyz 0 0 90))
+    )
+  )
   (dimension 60.325 (width 0.3) (layer Eco1.User)
     (gr_text "60,325 mm" (at 91.1225 109.935) (layer Eco1.User)
@@
   (segment (start 71.12 89.535) (end 72.39 88.265) (width 1.016) (layer F.Cu) (net 4))
   (segment (start 72.39 88.265) (end 72.39 85.725) (width 1.016) (layer F.Cu) (net 4))
-  (segment (start 78.74 82.55) (end 78.74 84.455) (width 1.016) (layer F.Cu) (net 5) (status 400000))
+  (segment (start 78.74 82.55) (end 78.74 84.455) (width 1.016) (layer F.Cu) (net 5))
   (segment (start 78.74 84.455) (end 80.01 85.725) (width 1.016) (layer F.Cu) (net 5))
   (segment (start 76.2 80.645) (end 78.105 80.645) (width 1.016) (layer F.Cu) (net 5))
-  (segment (start 78.74 81.28) (end 78.74 82.55) (width 1.016) (layer F.Cu) (net 5) (status 800000))
+  (segment (start 78.74 81.28) (end 78.74 82.55) (width 1.016) (layer F.Cu) (net 5))
   (segment (start 78.105 80.645) (end 78.74 81.28) (width 1.016) (layer F.Cu) (net 5))
   (segment (start 113.665 95.25) (end 117.475 95.25) (width 1.016) (layer F.Cu) (net 5))
