File: Hardware/_saved_rgb-strip.sch (KiCad schematic (older format))
At the start: 18 parts, among them CON1 BARREL_JACK, IC1 ATTINY84-P, P1 Bluetooth_Header, P2 CONN_01X03, Q1 HC49, SW1 SW_PUSH, U1 LM7805

Commit message: Created pcb layout
Parts:
- P3, P4: renamed from P?; footprint (none) -> Pin_Headers:Pin_Header_Straight_1x01
Changed lines of the file:
@@
 uC
 $Comp
-L CONN_01X01 P?
+L CONN_01X01 P4
 U 1 1 565EBF54
 P 4200 5950
-F 0 "P?" H 4200 6050 50  0000 C CNN
+F 0 "P4" H 4200 6050 50  0000 C CNN
 F 1 "CONN_01X01" V 4300 5950 50  0000 C CNN
-F 2 "" H 4200 5950 50  0000 C CNN
+F 2 "Pin_Headers:Pin_Header_Straight_1x01" H 4200 5950 50  0001 C CNN
 F 3 "" H 4200 5950 50  0000 C CNN
 	1    4200 5950
@@
 $EndComp
 $Comp
-L CONN_01X01 P?
+L CONN_01X01 P3
 U 1 1 565EC27F
 P 3600 5950
-F 0 "P?" H 3600 6050 50  0000 C CNN
+F 0 "P3" H 3600 6050 50  0000 C CNN
 F 1 "CONN_01X01" V 3700 5950 50  0000 C CNN
-F 2 "" H 3600 5950 50  0000 C CNN
+F 2 "Pin_Headers:Pin_Header_Straight_1x01" H 3600 5950 50  0001 C CNN
 F 3 "" H 3600 5950 50  0000 C CNN
 	1    3600 5950
