File: Hardware/rgb-strip.kicad_pcb (KiCad board)
At the start: 2 copper layers, 18 parts, among them CON1 BARREL_JACK, IC1 ATTINY84-P, P1 Bluetooth_Header, P2 CONN_01X03, P3 CONN_01X01, P4 CONN_01X01, Q1 HC49, SW1 SW_PUSH, U1 LM7805

Commit message: Finished board
Parts:
- removed D1, D2: LED, library:LED-3MM
- removed R2, R3: 330, Resistors_ThroughHole:Resistor_Horizontal_RM10mm
- added K1: CONN_3_V, Connect:bornier3, B.Cu at (113.7, 83.2)
- added LOGO_OSHW_silkscreen_5mm: val**, library:LOGO_OSHW_silkscreen_5mm, F.Cu at (73.7, 71.1)
- added P5: CONN_01X01, Pin_Headers:Pin_Header_Straight_1x01, B.Cu at (113.7, 74.3)
- added REF**: MountingHole_2-7mm, Mounting_Holes:MountingHole_2-7mm, B.Cu at (67.1, 71.1)
- added REF**: MountingHole_2-7mm, Mounting_Holes:MountingHole_2-7mm, B.Cu at (121.4, 100.1)
- added U2: ICSP, Pin_Headers:Pin_Header_Straight_2x03, B.Cu at (105.4, 77.5)
- P1: value Bluetooth_Header -> BT_Header-1x06; footprint Pin_Headers:Pin_Header_Angled_1x06 -> Pin_Headers:Pin_Header_Straight_1x06
- P2: value CONN_01X03 -> CONN_01X01; footprint Pin_Headers:Pin_Header_Straight_1x03 -> Pin_Headers:Pin_Header_Straight_1x01
- U1: value LM7805 -> 7805
- moved P3 21.0 mm to (87.0, 76.2)
- moved P2 15.3 mm to (122.4, 69.6), turned to 0 degrees
- moved P1 14.0 mm to (91.4, 72.4), turned to 90 degrees
- moved P4 7.65 mm to (87.0, 82.5)
- moved C3 5.08 mm to (83.8, 94.6), turned to 180 degrees
- moved U1 3.42 mm to (71.1, 82.5)
- moved C4 2.54 mm to (81.3, 82.5), turned to 180 degrees
- moved SW1 2.54 mm to (116.2, 100.3)
- moved R1 0.64 mm to (88.9, 86.4)
Connections:
- C3 pad 1: Net-(C3-Pad1) -> GND
- C3 pad 2: GND -> Net-(C3-Pad2)
- C4 pad 1: VCC -> GND
- C4 pad 2: GND -> VCC
- CON1 pad 1: Net-(C3-Pad1) -> Net-(C3-Pad2)
- IC1 pad 1: GND -> VCC
- IC1 pad 10: Net-(IC1-Pad10) -> BRX
- IC1 pad 11: Net-(IC1-Pad11) -> BTX
- IC1 pad 14: VCC -> GND
- IC1 pad 6: BTX -> MOSI
- IC1 pad 7: BRX -> Net-(IC1-Pad7)
- IC1 pad 8: PixelPin -> MISO
- IC1 pad 9: Net-(IC1-Pad9) -> SCK
- P2 pad 1: PixelPin -> GND
- U1 pad VI: Net-(C3-Pad1) -> Net-(C3-Pad2)
Routing:
- net BRX: track 27.1 -> 64.9 mm
- net BTX: track 36.3 -> 73.2 mm
- net SCK: track 0.00 -> 28.4 mm
- net Net-(C3-Pad2): track 0.00 -> 20.1 mm
- net Net-(C3-Pad1): track 16.0 -> 0.00 mm
- net MISO: track 0.00 -> 12.9 mm
- net RST: track 35.3 -> 48.0 mm
- net VCC: track 121.0 -> 133.6 mm
- net MOSI: track 0.00 -> 11.2 mm
- net PixelPin: track 7.62 -> 0.00 mm
- net Net-(D1-Pad2): track 5.87 -> 0.00 mm
- net Net-(D2-Pad2): track 5.08 -> 0.00 mm
Other:
- net class Default: clearance 0.53 -> 0.55
- net class PWR: clearance 0.53 -> 0.55
- rule trace_clearance: 0.53 -> 0.55
