File: Hardware/rgb-strip.sch (KiCad schematic (older format))
At the start: 18 parts, among them CON1 BARREL_JACK, IC1 ATTINY84-P, P1 Bluetooth_Header, P2 CONN_01X03, P3 CONN_01X01, P4 CONN_01X01, Q1 HC49, SW1 SW_PUSH, U1 LM7805

Commit message: Finished board
Parts:
- removed D1, D2: LED, library:LED-3MM, symbol LED
- removed P1: Bluetooth_Header, Pin_Headers:Pin_Header_Angled_1x06, symbol CONN_01X06
- removed P2: CONN_01X03, Pin_Headers:Pin_Header_Straight_1x03, symbol CONN_01X03
- removed R2, R3: 330, Resistors_ThroughHole:Resistor_Horizontal_RM10mm, symbol R
- removed U1: LM7805, library:LM7805, symbol LM7805
- added K1: CONN_3_V, Connect:bornier3, symbol CONN_3_V
- added P1: BT_Header-1x06, Pin_Headers:Pin_Header_Straight_1x06, symbol BT_Header-1x06
- added P2, P5: CONN_01X01, Pin_Headers:Pin_Header_Straight_1x01, symbol CONN_01X01
- added U1: 7805, library:LM7805, symbol 7805
- added U2: ICSP, Pin_Headers:Pin_Header_Straight_2x03, symbol ICSP
Connections:
- net BRX: now also IC1.10 ((PCINT3/T0/ADC3)PA3), P1.2 (RXD); no longer IC1.7 ((PCINT6/SDA/DI/MOSI/OC1A/ADC6)PA6)
- net BTX: now also IC1.11 ((PCINT2/AIN1/ADC2)PA2), P1.3 (TXD); no longer IC1.6 ((PCINT7/ICP/OC0B/ADC7)PA7)
- net GND: now also C3.1, C4.1, IC1.14 (GND), K1.1 (P1), P1.4 (GND), P2.1 (P1), P5.1 (P1), U1.GND, U2.6 (GND); no longer C3.2, C4.2, IC1.1 (VCC)
- net RST: now also U2.3 (RESET)
- net VCC: now also C4.2, IC1.1 (VCC), K1.3 (P3), P1.5 (Vcc), P1.6 (EN), U1.VO, U2.4 (VCC); no longer C4.1, IC1.14 (GND)
- net SCK: now reaches IC1.9 ((PCINT4/USCK/SCL/T1/ADC4)PA4)
- net SCK: now also U2.2 (SCK)
- net at CON1.1: now also C3.2, U1.VI; no longer C3.1
- net PixelPin renamed MISO
- net MISO: now also K1.2 (P2), U2.1 (MISO)
- new net MOSI: IC1.6 ((PCINT7/ICP/OC0B/ADC7)PA7), U2.5 (MOSI)
Other:
- note added: "ICSP Header"
- moved on the sheet: CON1, P3, P4
